File: Código Fuente/lab5.brd (EAGLE design)
At the start: 56.8 x 53.3 mm, 10 parts, among them P1 12V, P2 8V

Commit message: drb
Parts:
- removed Meter3, Meter5: (no value), AUTODESK_CIRCUITS_BREADBOARD:DC-POWER
- added Meter1: (no value), AUTODESK_CIRCUITS_BREADBOARD:DC-POWER
- added P3: 5.06V, AUTODESK_CIRCUITS_BREADBOARD:2P-2.54-65/35MIL
- added R6: 1k‎Ω, AUTODESK_CIRCUITS_BREADBOARD:0207/10
- added R7: 100‎Ω, AUTODESK_CIRCUITS_BREADBOARD:0207/10
- P1: value 12V -> 2V
- P2: value 8V -> 12V
- R1: value 1.8k‎Ω -> 560‎Ω
- R2: value 470‎Ω -> 4.7k‎Ω
- R3: value 1.5k‎Ω -> 299‎Ω
- R4: value 2.2k‎Ω -> 1k‎Ω
- R5: value 3.9k‎Ω -> 330‎Ω
- moved R4 63.5 mm to (5.00, 111.7)
- moved R3 63.5 mm to (5.00, 99.0)
- moved Meter2 50.8 mm to (5.00, 149.8)
- moved R5 25.4 mm to (5.00, 35.5)
Connections:
- new net N$6: P1.1, R1.1, R2.2
- new net N$7: R6.2, R7.2
- new net N$8: P1.2, R5.2, R7.1
- new net N$9: P2.1, R2.1, R5.1, R6.1
- net N$1: now also Meter1.+, R3.2; no longer Meter5.+, R1.2, R2.2, R4.2
- net N$2: now also P3.2, R3.1; no longer P1.2, R1.1
- net N$3: now also Meter1.-, Meter2.+, R4.2; no longer P2.2, R3.2
- net N$4: now also P3.1, R4.1; no longer Meter2.+, Meter3.-, Meter5.-, P1.1, P2.1, R2.1, R5.1
- net N$5: now also P2.2, R1.2; no longer Meter3.+, R3.1, R4.1, R5.2
Changed lines of the file:
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@@
 </autorouter>
 <elements>
-<element value="1.8k‎Ω" name="R1" library="AUTODESK_CIRCUITS_BREADBOARD" package="0207/10" x="5" y="10.08"></element><element value="470‎Ω" name="R2" library="AUTODESK_CIRCUITS_BREADBOARD" package="0207/10" x="5" y="22.78"></element><element value="1.5k‎Ω" name="R3" library="AUTODESK_CIRCUITS_BREADBOARD" package="0207/10" x="5" y="35.480000000000004"></element><element value="2.2k‎Ω" name="R4" library="AUTODESK_CIRCUITS_BREADBOARD" package="0207/10" x="5" y="48.18"></element><element value="3.9k‎Ω" name="R5" library="AUTODESK_CIRCUITS_BREADBOARD" package="0207/10" x="5" y="60.879999999999995"></element><element value="12V" name="P1" library="AUTODESK_CIRCUITS_BREADBOARD" package="2P-2.54-65/35MIL" x="5" y="73.58"></element><element value="8V" name="P2" library="AUTODESK_CIRCUITS_BREADBOARD" package="2P-2.54-65/35MIL" x="5" y="86.28"></element><element value="" name="Meter2" library="AUTODESK_CIRCUITS_BREADBOARD" package="DC-POWER" x="5" y="98.98"></element><element value="" name="Meter3" library="AUTODESK_CIRCUITS_BREADBOARD" package="DC-POWER" x="5" y="111.68"></element><element value="" name="Meter5" library="AUTODESK_CIRCUITS_BREADBOARD" package="DC-POWER" x="5" y="124.38000000000001"></element></elements>
+<element value="560‎Ω" name="R1" library="AUTODESK_CIRCUITS_BREADBOARD" package="0207/10" x="5" y="10.08"></element><element value="4.7k‎Ω" name="R2" library="AUTODESK_CIRCUITS_BREADBOARD" package="0207/10" x="5" y="22.78"></element><element value="330‎Ω" name="R5" library="AUTODESK_CIRCUITS_BREADBOARD" package="0207/10" x="5" y="35.480000000000004"></element><element value="1k‎Ω" name="R6" library="AUTODESK_CIRCUITS_BREADBOARD" package="0207/10" x="5" y="48.18"></element><element value="100‎Ω" name="R7" library="AUTODESK_CIRCUITS_BREADBOARD" package="0207/10" x="5" y="60.879999999999995"></element><element value="2V" name="P1" library="AUTODESK_CIRCUITS_BREADBOARD" package="2P-2.54-65/35MIL" x="5" y="73.58"></element><element value="12V" name="P2" library="AUTODESK_CIRCUITS_BREADBOARD" package="2P-2.54-65/35MIL" x="5" y="86.28"></element><element value="299‎Ω" name="R3" library="AUTODESK_CIRCUITS_BREADBOARD" package="0207/10" x="5" y="98.98"></element><element value="1k‎Ω" name="R4" library="AUTODESK_CIRCUITS_BREADBOARD" package="0207/10" x="5" y="111.68"></element><element value="5.06V" name="P3" library="AUTODESK_CIRCUITS_BREADBOARD" package="2P-2.54-65/35MIL" x="5" y="124.38000000000001"></element><element value="" name="Meter1" library="AUTODESK_CIRCUITS_BREADBOARD" package="DC-POWER" x="5" y="137.08"></element><element value="" name="Meter2" library="AUTODESK_CIRCUITS_BREADBOARD" package="DC-POWER" x="5" y="149.78000000000003"></element></elements>
 <signals>
-<signal name="N$1"><contactref element="R1" pad="2"></contactref><contactref element="R4" pad="2"></contactref><wire x1="10.08" y1="10.08" x2="10.08" y2="48.18" width="0" layer="19" extent="1-1"></wire><contactref element="Meter5" pad="+"></contactref><wire x1="10.08" y1="48.18" x2="5" y2="126.92000000000002" width="0" layer="19" extent="1-1"></wire><contactref element="R2" pad="2"></contactref><wire x1="5" y1="126.92000000000002" x2="10.08" y2="22.78" width="0" layer="19" extent="1-1"></wire></signal><signal name="N$2"><contactref element="R1" pad="1"></contactref><contactref element="P1" pad="2"></contactref><wire x1="-0.08000000000000007" y1="10.08" x2="5" y2="72.31" width="0" layer="19" extent="1-1"></wire></signal><signal name="N$3"><contactref element="P2" pad="2"></contactref><contactref element="R3" pad="2"></contactref><wire x1="5" y1="85.01" x2="10.08" y2="35.480000000000004" width="0" layer="19" extent="1-1"></wire></signal><signal name="N$4"><contactref element="P1" pad="1"></contactref><contactref element="Meter2" pad="+"></contactref><wire x1="5" y1="74.85" x2="5" y2="101.52000000000001" width="0" layer="19" extent="1-1"></wire><contactref element="R2" pad="1"></contactref><wire x1="5" y1="101.52000000000001" x2="-0.08000000000000007" y2="22.78" width="0" layer="19" extent="1-1"></wire><contactref element="Meter3" pad="-"></contactref><wire x1="-0.08000000000000007" y1="22.78" x2="5" y2="109.14" width="0" layer="19" extent="1-1"></wire><contactref element="P2" pad="1"></contactref><wire x1="5" y1="109.14" x2="5" y2="87.55" width="0" layer="19" extent="1-1"></wire><contactref element="Meter2" pad="-"></contactref><wire x1="5" y1="87.55" x2="5" y2="96.44" width="0" layer="19" extent="1-1"></wire><contactref element="Meter5" pad="-"></contactref><wire x1="5" y1="96.44" x2="5" y2="121.84" width="0" layer="19" extent="1-1"></wire><contactref element="R5" pad="1"></contactref><wire x1="5" y1="121.84" x2="-0.08000000000000007" y2="60.879999999999995" width="0" layer="19" extent="1-1"></wire></signal><signal name="N$5"><contactref element="R4" pad="1"></contactref><contactref element="Meter3" pad="+"></contactref><wire x1="-0.08000000000000007" y1="48.18" x2="5" y2="114.22000000000001" width="0" layer="19" extent="1-1"></wire><contactref element="R3" pad="1"></contactref><wire x1="5" y1="114.22000000000001" x2="-0.08000000000000007" y2="35.480000000000004" width="0" layer="19" extent="1-1"></wire><contactref element="R5" pad="2"></contactref><wire x1="-0.08000000000000007" y1="35.480000000000004" x2="10.08" y2="60.879999999999995" width="0" layer="19" extent="1-1"></wire></signal></signals>
+<signal name="N$1"><contactref element="R3" pad="2"></contactref><contactref element="Meter1" pad="+"></contactref><wire x1="10.08" y1="98.98" x2="5" y2="139.62" width="0" layer="19" extent="1-1"></wire></signal><signal name="N$2"><contactref element="P3" pad="2"></contactref><contactref element="R3" pad="1"></contactref><wire x1="5" y1="123.11000000000001" x2="-0.08000000000000007" y2="98.98" width="0" layer="19" extent="1-1"></wire></signal><signal name="N$3"><contactref element="R4" pad="2"></contactref><contactref element="Meter1" pad="-"></contactref><wire x1="10.08" y1="111.68" x2="5" y2="134.54000000000002" width="0" layer="19" extent="1-1"></wire><contactref element="Meter2" pad="+"></contactref><wire x1="5" y1="134.54000000000002" x2="5" y2="152.32000000000002" width="0" layer="19" extent="1-1"></wire></signal><signal name="N$4"><contactref element="R4" pad="1"></contactref><contactref element="Meter2" pad="-"></contactref><wire x1="-0.08000000000000007" y1="111.68" x2="5" y2="147.24000000000004" width="0" layer="19" extent="1-1"></wire><contactref element="P3" pad="1"></contactref><wire x1="5" y1="147.24000000000004" x2="5" y2="125.65" width="0" layer="19" extent="1-1"></wire></signal><signal name="N$5"><contactref element="P2" pad="2"></contactref><contactref element="R1" pad="2"></contactref><wire x1="5" y1="85.01" x2="10.08" y2="10.08" width="0" layer="19" extent="1-1"></wire></signal><signal name="N$6"><contactref element="R2" pad="2"></contactref><contactref element="P1" pad="1"></contactref><wire x1="10.08" y1="22.78" x2="5" y2="74.85" width="0" layer="19" extent="1-1"></wire><contactref element="R1" pad="1"></contactref><wire x1="5" y1="74.85" x2="-0.08000000000000007" y2="10.08" width="0" layer="19" extent="1-1"></wire></signal><signal name="N$7"><contactref element="R7" pad="2"></contactref><contactref element="R6" pad="2"></contactref><wire x1="10.08" y1="60.879999999999995" x2="10.08" y2="48.18" width="0" layer="19" extent="1-1"></wire></signal><signal name="N$8"><contactref element="R7" pad="1"></contactref><contactref element="R5" pad="2"></contactref><wire x1="-0.08000000000000007" y1="60.879999999999995" x2="10.08" y2="35.480000000000004" width="0" layer="19" extent="1-1"></wire><contactref element="P1" pad="2"></contactref><wire x1="10.08" y1="35.480000000000004" x2="5" y2="72.31" width="0" layer="19" extent="1-1"></wire></signal><signal name="N$9"><contactref element="R6" pad="1"></contactref><contactref element="R2" pad="1"></contactref><wire x1="-0.08000000000000007" y1="48.18" x2="-0.08000000000000007" y2="22.78" width="0" layer="19" extent="1-1"></wire><contactref element="R5" pad="1"></contactref><wire x1="-0.08000000000000007" y1="22.78" x2="-0.08000000000000007" y2="35.480000000000004" width="0" layer="19" extent="1-1"></wire><contactref element="P2" pad="1"></contactref><wire x1="-0.08000000000000007" y1="35.480000000000004" x2="5" y2="87.55" width="0" layer="19" extent="1-1"></wire></signal></signals>
 </board>
 </drawing>
